File: hardware/Interconnexions/interconnexions.sch (EAGLE design)
At the start: 102 parts, among them K5 ZNS5106

Commit message: 1 carte. 3 strap.
Parts:
- removed 24V_BATT: (no value), con-amp:MTA02-156
- removed C17, C18: (no value), resistor:CPOL-EUE2,5-6E
- added AX12-7, AX12-8: (no value), con-amp:MTA03-100
- added BORNIER_LI-PO: (no value), con-ptr500:AK300/2
- ARRET_URGENCE, BORNIER_MONTE-PLOT, BORNIER_MOTEUR_DROIT, BORNIER_MOTEUR_GAUCHE, BUZZER, BYPASS_RELAI: device con-amp:MTA02-156 -> con-ptr500:AK300/2
- D1, D2, D3, D4: value 1N4728 -> (none); device diode:1N4728 -> diode:ZENER-DIODEZD-2.5
- LED1: value (none) -> RED
- LED2: value (none) -> GREEN half
- LED3: value (none) -> GREEN full
- MD-PD-PWM, MG-PD-PWM, MP-PD-PWM: device rcl:R-EU_0207/7 -> resistor:R-EU_0207/7
- MD-PU-PWM, MG-PU-PWM, MP-PU-PWM: device rcl:R-EU_0207/7 -> resistor:R-EU_0207/15
- R3, R5, R6, R8: device resistor:R-EU_0204/7 -> resistor:R-EU_0207/2V
Connections:
- removed net N$22: 24V_BATT.1, DIODE24V.A
- new net N$38: ARRET_URGENCE-2.KL, DIODE24V.A
- net +24V: now also BYPASS_RELAI-2.KL; no longer BYPASS_RELAI.2
- net +24V_BATT: now also BYPASS_RELAI-1.KL, DIODE24V.C; no longer ARRET_URGENCE.1, BYPASS_RELAI.1
- net +9V: now also AX12-7.2, AX12-8.2; no longer C17.+, C18.+
- net GND: now also AX12-7.1, AX12-8.1, BORNIER_LI-PO-1.KL, BUZZER-2.KL; no longer 24V_BATT.2, BUZZER.1, C17.-, C18.-
- net MONTE-PLOT_DIR: now also U$1.PD14; no longer U$1.PD10
- net MOTEUR_DROIT-DIR: now also U$1.PD12; no longer U$1.PD14
- net MOTEUR_DROIT-PWM: now also U$1.PC6; no longer U$1.PC7
- net MOTEUR_GAUCHE-DIR: now also U$1.PD10; no longer U$1.PD12
- net MOTEUR_GAUCHE-PWM: now also U$1.PC7; no longer U$1.PC6
- net N$10: now also BORNIER_MOTEUR_DROIT-1.KL; no longer BORNIER_MOTEUR_DROIT.1
- net N$11: now also BORNIER_MOTEUR_GAUCHE-1.KL; no longer BORNIER_MOTEUR_GAUCHE.1
- net N$12: now also BORNIER_MOTEUR_GAUCHE-2.KL; no longer BORNIER_MOTEUR_GAUCHE.2
- net N$18: now also BORNIER_MONTE-PLOT-1.KL; no longer BORNIER_MONTE-PLOT.1
- net N$19: now also BORNIER_MONTE-PLOT-2.KL; no longer BORNIER_MONTE-PLOT.2
- net N$23: now also ARRET_URGENCE-1.KL, BORNIER_LI-PO-2.KL; no longer ARRET_URGENCE.2, DIODE24V.C
- net N$28: now also BUZZER-1.KL; no longer BUZZER.2
- net N$9: now also BORNIER_MOTEUR_DROIT-2.KL; no longer BORNIER_MOTEUR_DROIT.2
- net UART_AX12: now also AX12-7.3, AX12-8.3
Other:
- note added: "DIR MONTE-PLOT PD14"
- note added: "DIR MOTEUR DROIT PD12"
- note added: "DIR MOTEUR GAUCHE PD10"
- note added: "PWM MONTE-PLOT PC8"
- note added: "PWM MOTEUR DROIT PC6"
- note added: "PWM MOTEUR GAUCHE PC7"
- note removed: "DIR MOTEUR DROIT PD14"
- note removed: "DIR MOTEUR GAUCHE PD12"
- note removed: "PWM MOTEUR DROIT PC7"
- note removed: "PWM MOTEUR GAUCHE PC6"
- moved on the sheet: AX12-1, AX12-2, AX12-3, AX12-4, AX12-5, AX12-6, C1, C10, C2, C3, C4, C5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

Commit message: Carte : modification de la distance interpistes
Parts:
- D5: value 1N4933 -> (none); device diode:1N4933 -> diode:DIODE-D-2.5
- MD-PD-DIR, MP-PD-DIR: device rcl:R-EU_0207/7 -> rcl:R-EU_0207/10
- R1: device resistor:R-EU_0204/7 -> rcl:R-EU_0207/2V
- R8: device resistor:R-EU_0207/2V -> rcl:R-EU_0204/5
Connections:
- net CAPTEUR_4: now also U$1.PC11; no longer U$1.PA15
- net CAPTEUR_A1: now also U$1.PA6; no longer U$1.PC1
- net CAPTEUR_A2: now also U$1.PA4; no longer U$1.PC3
- net CODDROITB: now also U$1.PB4; no longer U$1.PC11
- net GND: now also U$1.PA10, U$1.PA13, U$1.PB2, U$1.PE2, U$1.PE3; no longer U$1.GND8
Changed lines of the file:
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@@
 <?xml version="1.0" encoding="utf-8"?>
 <!DOCTYPE eagle SYSTEM "eagle.dtd">
-<eagle version="6.3">
+<eagle version="7.2.0">
 <drawing>
 <settings>
@@
 <part name="MD-PU-PWM" library="resistor" deviceset="R-EU_" device="0207/15" value="100"/>
 <part name="MD-PD-PWM" library="resistor" deviceset="R-EU_" device="0207/7" value="3.3k"/>
-<part name="MD-PD-DIR" library="rcl" deviceset="R-EU_" device="0207/7" value="3.3k"/>
+<part name="MD-PD-DIR" library="rcl" deviceset="R-EU_" device="0207/10" value="3.3k"/>
 <part name="SUPPLY23" library="supply2" deviceset="GND" device=""/>
 <part name="C8" library="rcl" deviceset="CPOL-EU" device="E3.5-8" value="1µF"/>
@@
 <part name="MP-PU-PWM" library="resistor" deviceset="R-EU_" device="0207/15" value="100"/>
 <part name="MP-PD-PWM" library="resistor" deviceset="R-EU_" device="0207/7" value="3.3k"/>
-<part name="MP-PD-DIR" library="rcl" deviceset="R-EU_" device="0207/7" value="3.3k"/>
+<part name="MP-PD-DIR" library="rcl" deviceset="R-EU_" device="0207/10" value="3.3k"/>
 <part name="SUPPLY27" library="supply2" deviceset="GND" device=""/>
 <part name="C11" library="rcl" deviceset="CPOL-EU" device="E3.5-8" value="1µF"/>
@@
 <part name="D1" library="diode" deviceset="ZENER-DIODE" device="ZD-2.5"/>
 <part name="T1" library="transistor" deviceset="*-NPN-" device="TO92-CBE" technology="2N5400"/>
-<part name="R1" library="resistor" deviceset="R-EU_" device="0204/7"/>
+<part name="R1" library="rcl" deviceset="R-EU_" device="0207/2V"/>
 <part name="R2" library="resistor" deviceset="R-EU_" device="0204/7"/>
 <part name="R3" library="resistor" deviceset="R-EU_" device="0207/2V"/>
@@
 <part name="R7" library="resistor" deviceset="R-EU_" device="0204/7"/>
 <part name="T4" library="transistor" deviceset="*-NPN-" device="TO92-CBE" technology="2N5400"/>
-<part name="R8" library="resistor" deviceset="R-EU_" device="0207/2V"/>
+<part name="R8" library="rcl" deviceset="R-EU_" device="0204/5"/>
 <part name="SUPPLY69" library="supply2" deviceset="GND" device=""/>
 <part name="LED1" library="led" deviceset="LED" device="5MM" value="RED"/>
@@
 <part name="LED3" library="led" deviceset="LED" device="5MM" value="GREEN full"/>
 <part name="SUPPLY70" library="supply2" deviceset="+5V" device=""/>
-<part name="D5" library="diode" deviceset="1N4933" device=""/>
+<part name="D5" library="diode" deviceset="DIODE-" device="D-2.5"/>
 <part name="SUPPLY71" library="supply2" deviceset="GND" device=""/>
 <part name="SUPPLY72" library="supply2" deviceset="GND" device=""/>
@@
 <instance part="LED3" gate="G$1" x="171.45" y="-223.52"/>
 <instance part="SUPPLY70" gate="+5V" x="133.35" y="-193.04" rot="R90"/>
-<instance part="D5" gate="1" x="198.12" y="-167.64" rot="R180"/>
+<instance part="D5" gate="G$1" x="198.12" y="-167.64" rot="R180"/>
 <instance part="SUPPLY71" gate="GND" x="158.75" y="-189.23" rot="R270"/>
 <instance part="SUPPLY72" gate="GND" x="156.21" y="-203.2" rot="R270"/>
@@
 </segment>
 <segment>
-<pinref part="U$1" gate="G$1" pin="GND8"/>
-<wire x1="81.28" y1="2.54" x2="76.2" y2="2.54" width="0.1524" layer="91"/>
-<label x="76.2" y="2.54" size="1.778" layer="95"/>
-</segment>
-<segment>
 <pinref part="U$1" gate="G$1" pin="GND9"/>
 <wire x1="111.76" y1="2.54" x2="116.84" y2="2.54" width="0.1524" layer="91"/>
@@
 <pinref part="SUPPLY72" gate="GND" pin="GND"/>
 </segment>
+<segment>
+<pinref part="U$1" gate="G$1" pin="PE3"/>
+<wire x1="111.76" y1="45.72" x2="116.84" y2="45.72" width="0.1524" layer="91"/>
+<label x="111.76" y="45.72" size="1.778" layer="95"/>
+</segment>
+<segment>
+<pinref part="U$1" gate="G$1" pin="PE2"/>
+<wire x1="81.28" y1="45.72" x2="76.2" y2="45.72" width="0.1524" layer="91"/>
+<label x="76.2" y="45.72" size="1.778" layer="95"/>
+</segment>
+<segment>
+<pinref part="U$1" gate="G$1" pin="PA13"/>
+<wire x1="111.76" y1="12.7" x2="116.84" y2="12.7" width="0.1524" layer="91"/>
+<label x="116.84" y="12.7" size="1.778" layer="95"/>
+</segment>
+<segment>
+<pinref part="U$1" gate="G$1" pin="PA10"/>
+<wire x1="81.28" y1="12.7" x2="76.2" y2="12.7" width="0.1524" layer="91"/>
+<label x="76.2" y="12.7" size="1.778" layer="95"/>
+</segment>
+<segment>
+<pinref part="U$1" gate="G$1" pin="PB2"/>
+<wire x1="25.4" y1="35.56" x2="30.48" y2="35.56" width="0.1524" layer="91"/>
+<label x="30.48" y="35.56" size="1.778" layer="95"/>
+</segment>
 </net>
 <net name="+24V" class="0">
@@
 </segment>
 <segment>
-<pinref part="U$1" gate="G$1" pin="PC11"/>
-<wire x1="111.76" y1="17.78" x2="116.84" y2="17.78" width="0.1524" layer="91"/>
-<label x="116.84" y="17.78" size="1.778" layer="95"/>
+<pinref part="U$1" gate="G$1" pin="PB4"/>
+<wire x1="81.28" y1="33.02" x2="73.66" y2="33.02" width="0.1524" layer="91"/>
+<label x="63.5" y="33.02" size="1.778" layer="95"/>
 </segment>
 </net>
@@
 </segment>
 <segment>
-<pinref part="U$1" gate="G$1" pin="PA15"/>
-<wire x1="111.76" y1="15.24" x2="116.84" y2="15.24" width="0.1524" layer="91"/>
-<label x="116.84" y="15.24" size="1.778" layer="95"/>
+<pinref part="U$1" gate="G$1" pin="PC11"/>
+<wire x1="111.76" y1="17.78" x2="116.84" y2="17.78" width="0.1524" layer="91"/>
+<label x="116.84" y="17.78" size="1.778" layer="95"/>
 </segment>
 </net>
@@
 </segment>
 <segment>
-<pinref part="U$1" gate="G$1" pin="PC1"/>
-<wire x1="-5.08" y1="55.88" x2="-10.16" y2="55.88" width="0.1524" layer="91"/>
-<label x="-20.32" y="55.88" size="1.778" layer="95"/>
+<pinref part="U$1" gate="G$1" pin="PA6"/>
+<wire x1="25.4" y1="43.18" x2="30.48" y2="43.18" width="0.1524" layer="91"/>
+<label x="30.48" y="43.18" size="1.778" layer="95"/>
 </segment>
 </net>
@@
 </segment>
 <segment>
-<pinref part="U$1" gate="G$1" pin="PC3"/>
-<wire x1="-5.08" y1="53.34" x2="-10.16" y2="53.34" width="0.1524" layer="91"/>
-<label x="-20.32" y="53.34" size="1.778" layer="95"/>
+<pinref part="U$1" gate="G$1" pin="PA4"/>
+<wire x1="25.4" y1="45.72" x2="30.48" y2="45.72" width="0.1524" layer="91"/>
+<label x="30.48" y="45.72" size="1.778" layer="95"/>
 </segment>
 </net>
@@
 <wire x1="193.04" y1="-161.29" x2="189.23" y2="-161.29" width="0.1524" layer="91"/>
 <junction x="189.23" y="-161.29"/>
-<pinref part="D5" gate="1" pin="C"/>
+<pinref part="D5" gate="G$1" pin="C"/>
 <wire x1="195.58" y1="-167.64" x2="189.23" y2="-167.64" width="0.1524" layer="91"/>
 <junction x="189.23" y="-167.64"/>
@@
 <wire x1="203.2" y1="-161.29" x2="207.01" y2="-161.29" width="0.1524" layer="91"/>
 <wire x1="207.01" y1="-161.29" x2="207.01" y2="-167.64" width="0.1524" layer="91"/>
-<pinref part="D5" gate="1" pin="A"/>
+<pinref part="D5" gate="G$1" pin="A"/>
 <wire x1="207.01" y1="-167.64" x2="207.01" y2="-176.53" width="0.1524" layer="91"/>
 <wire x1="200.66" y1="-167.64" x2="207.01" y2="-167.64" width="0.1524" layer="91"/>

Commit message: Carte d'interconnexions fonctionnelle
Parts:
- added LED4: GREEN, led:LED5MM
- added R10: 1k, rcl:R-EU_0207/2V
Connections:
- new net N$22: LED4.C, R10.2
- net +5V: now also LED4.A
- net GND: now also R10.1
Changed lines of the file:
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@@
 <?xml version="1.0" encoding="utf-8"?>
 <!DOCTYPE eagle SYSTEM "eagle.dtd">
-<eagle version="7.2.0">
+<eagle version="6.3">
 <drawing>
 <settings>
@@
 <setting verticaltext="up"/>
 </settings>
-<grid distance="0.1" unitdist="inch" unit="inch" style="lines" multiple="1" display="no" altdistance="0.01" altunitdist="inch" altunit="inch"/>
+<grid distance="0.1" unitdist="inch" unit="inch" style="lines" multiple="1" display="no" altdistance="0.05" altunitdist="inch" altunit="inch"/>
 <layers>
 <layer number="1" name="Top" color="4" fill="1" visible="no" active="no"/>
@@
 <part name="AX12-7" library="con-amp" deviceset="MTA03-100" device=""/>
 <part name="AX12-8" library="con-amp" deviceset="MTA03-100" device=""/>
+<part name="SUPPLY74" library="supply2" deviceset="GND" device=""/>
+<part name="R10" library="rcl" deviceset="R-EU_" device="0207/2V" value="1k"/>
+<part name="LED4" library="led" deviceset="LED" device="5MM" value="GREEN"/>
+<part name="SUPPLY73" library="supply2" deviceset="+5V" device=""/>
 </parts>
 <sheets>
@@
 <instance part="AX12-7" gate="G$1" x="182.88" y="15.24"/>
 <instance part="AX12-8" gate="G$1" x="182.88" y="7.62"/>
+<instance part="SUPPLY74" gate="GND" x="271.78" y="-139.7" rot="R90"/>
+<instance part="R10" gate="G$1" x="261.62" y="-139.7" rot="R180"/>
+<instance part="LED4" gate="G$1" x="248.92" y="-139.7" rot="R90"/>
+<instance part="SUPPLY73" gate="+5V" x="241.3" y="-139.7" rot="R90"/>
 </instances>
 <busses>
@@
 <label x="30.48" y="35.56" size="1.778" layer="95"/>
 </segment>
+<segment>
+<pinref part="R10" gate="G$1" pin="1"/>
+<pinref part="SUPPLY74" gate="GND" pin="GND"/>
+<wire x1="266.7" y1="-139.7" x2="269.24" y2="-139.7" width="0.1524" layer="91"/>
+</segment>
 </net>
 <net name="+24V" class="0">
@@
 <pinref part="R7" gate="G$1" pin="1"/>
 <pinref part="SUPPLY70" gate="+5V" pin="+5V"/>
+</segment>
+<segment>
+<pinref part="SUPPLY73" gate="+5V" pin="+5V"/>
+<pinref part="LED4" gate="G$1" pin="A"/>
+<wire x1="243.84" y1="-139.7" x2="246.38" y2="-139.7" width="0.1524" layer="91"/>
 </segment>
 </net>
@@
 </segment>
 </net>
+<net name="N$22" class="0">
+<segment>
+<pinref part="LED4" gate="G$1" pin="C"/>
+<pinref part="R10" gate="G$1" pin="2"/>
+<wire x1="254" y1="-139.7" x2="256.54" y2="-139.7" width="0.1524" layer="91"/>
+</segment>
+</net>

Commit message: documentation carte d'interconnexions
Parts:
- R10: value 1k -> 270
Changed lines of the file:
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@@
 <setting verticaltext="up"/>
 </settings>
-<grid distance="0.1" unitdist="inch" unit="inch" style="lines" multiple="1" display="no" altdistance="0.05" altunitdist="inch" altunit="inch"/>
+<grid distance="0.1" unitdist="inch" unit="inch" style="lines" multiple="1" display="no" altdistance="0.01" altunitdist="inch" altunit="inch"/>
 <layers>
 <layer number="1" name="Top" color="4" fill="1" visible="no" active="no"/>
@@
 <part name="AX12-8" library="con-amp" deviceset="MTA03-100" device=""/>
 <part name="SUPPLY74" library="supply2" deviceset="GND" device=""/>
-<part name="R10" library="rcl" deviceset="R-EU_" device="0207/2V" value="1k"/>
+<part name="R10" library="rcl" deviceset="R-EU_" device="0207/2V" value="270"/>
 <part name="LED4" library="led" deviceset="LED" device="5MM" value="GREEN"/>
 <part name="SUPPLY73" library="supply2" deviceset="+5V" device=""/>

Commit message: maj doc cartes elec
Connections:
- net CAPTEUR_A1 renamed CAPTEUR_A1_US
- net CAPTEUR_A3 renamed CAPTEUR_A3_US
- net CAPTEUR_A4 renamed CAPTEUR_A4_US
- net CAPTEUR_A6 renamed CAPTEUR_A6_US
Changed lines of the file:
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@@
 </segment>
 </net>
-<net name="CAPTEUR_A1" class="0">
+<net name="CAPTEUR_A1_US" class="0">
 <segment>
 <pinref part="JP2" gate="A" pin="3"/>
@@
 </segment>
 </net>
-<net name="CAPTEUR_A3" class="0">
+<net name="CAPTEUR_A3_US" class="0">
 <segment>
 <pinref part="JP3" gate="A" pin="3"/>
@@
 </segment>
 </net>
-<net name="CAPTEUR_A4" class="0">
+<net name="CAPTEUR_A4_US" class="0">
 <segment>
 <pinref part="JP4" gate="A" pin="3"/>
@@
 </segment>
 </net>
-<net name="CAPTEUR_A6" class="0">
+<net name="CAPTEUR_A6_US" class="0">
 <segment>
 <pinref part="JP6" gate="A" pin="3"/>

Commit message: maj doc hardware
Connections:
- net CAPTEUR_A1_US renamed CAPTEUR_US_AV_D
- net CAPTEUR_A4_US renamed CAPTEUR_US_AR_D
- net CAPTEUR_A5 renamed CAPTEUR_A1
- net CAPTEUR_A6_US renamed CAPTEUR_US_AR_G
- removed net CAPTEUR_A3_US: JP3.3, U$1.PA5
- new net CAPTEUR_US_AV_G: JP1.3, U$1.PA4
- net CAPTEUR_1: now also JP16.3, U$1.PC11; no longer JP13.3, U$1.PD6
- net CAPTEUR_2: now also JP15.3, U$1.PD0; no longer JP14.3, U$1.PD2
- net CAPTEUR_3: now also JP14.3, U$1.PD2; no longer JP15.3, U$1.PD0
- net CAPTEUR_4: now also JP13.3, U$1.PD6; no longer JP16.3, U$1.PC11
- net CAPTEUR_A2: now also JP3.3, U$1.PA5; no longer JP1.3, U$1.PA4
Changed lines of the file:
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@@
 </segment>
 </net>
-<net name="CAPTEUR_1" class="0">
+<net name="CAPTEUR_4" class="0">
 <segment>
 <pinref part="JP13" gate="A" pin="3"/>
@@
 </segment>
 </net>
-<net name="CAPTEUR_2" class="0">
+<net name="CAPTEUR_3" class="0">
 <segment>
 <pinref part="JP14" gate="A" pin="3"/>
@@
 </segment>
 </net>
-<net name="CAPTEUR_3" class="0">
+<net name="CAPTEUR_2" class="0">
 <segment>
 <pinref part="JP15" gate="A" pin="3"/>
@@
 </segment>
 </net>
-<net name="CAPTEUR_4" class="0">
+<net name="CAPTEUR_1" class="0">
 <segment>
 <pinref part="JP16" gate="A" pin="3"/>
@@
 </segment>
 </net>
-<net name="CAPTEUR_A1_US" class="0">
+<net name="CAPTEUR_US_AV_D" class="0">
 <segment>
 <pinref part="JP2" gate="A" pin="3"/>
@@
 </segment>
 </net>
-<net name="CAPTEUR_A2" class="0">
+<net name="CAPTEUR_US_AV_G" class="0">
 <segment>
 <pinref part="JP1" gate="A" pin="3"/>
@@
 </segment>
 </net>
-<net name="CAPTEUR_A3_US" class="0">
+<net name="CAPTEUR_A2" class="0">
 <segment>
 <pinref part="JP3" gate="A" pin="3"/>
@@
 </segment>
 </net>
-<net name="CAPTEUR_A5" class="0">
+<net name="CAPTEUR_A1" class="0">
 <segment>
 <pinref part="JP5" gate="A" pin="3"/>
@@
 </segment>
 </net>
-<net name="CAPTEUR_A4_US" class="0">
+<net name="CAPTEUR_US_AR_D" class="0">
 <segment>
 <pinref part="JP4" gate="A" pin="3"/>
@@
 <pinref part="U$1" gate="G$1" pin="PA7"/>
 <wire x1="-5.08" y1="43.18" x2="-10.16" y2="43.18" width="0.1524" layer="91"/>
-<label x="-20.32" y="43.18" size="1.778" layer="95"/>
+<label x="-27.94" y="43.18" size="1.778" layer="95"/>
 </segment>
 </net>
-<net name="CAPTEUR_A6_US" class="0">
+<net name="CAPTEUR_US_AR_G" class="0">
 <segment>
 <pinref part="JP6" gate="A" pin="3"/>
@@
 <pinref part="U$1" gate="G$1" pin="PB1"/>
 <wire x1="-5.08" y1="38.1" x2="-10.16" y2="38.1" width="0.1524" layer="91"/>
-<label x="-20.32" y="38.1" size="1.778" layer="95"/>
+<label x="-27.94" y="38.1" size="1.778" layer="95"/>
 </segment>
 </net>
