File: hardware/Robot secondaire/robot secondaire.sch (EAGLE design)
At the start: 27 parts, among them IC1 7812TV

Commit message: maj elec robot secondaire
Parts:
- added JP22: (no value), pinhead:PINHD-1X3
- added TX: (no value), pinhead:PINHD-1X1
- IC1: value 7812TV -> 7812T; device linear:7812TV -> linear:7812T
- renumbered JP14 to 8, JP15 to 9, JP16 to A0, JP17 to GND, JP5 to A02, JP6 to RAW, JP7 to VCC
Connections:
- net N$9 renamed CMD_MOTEUR
- removed net N$10: JP20.2, JP21.1
- new net +9V: JP20.2, JP21.1, JP22.2
- new net AX12: JP22.1, TX.1
- net +12V: now also C3.+; no longer C3.-
- net GND: now also C3.-, JP22.3; no longer C3.+
Other:
- moved on the sheet: C3
